Commit message: using new panda model with pan attached

File: CS141 Final Project/Panda_Juggling/resources/franka_description/robots/hand.xacro (robot description, xacro)
@@ -21,44 +21,77 @@
       </collision>
     </link>
-    <link name="${ns}_leftfinger">
-      <visual>
-        <geometry>
-          <mesh filename="package://franka_description/meshes/visual/finger.dae"/>
-        </geometry>
-      </visual>
-      <collision>
-        <geometry>
-          <mesh filename="package://franka_description/meshes/collision/finger.stl"/>
-        </geometry>
-      </collision>
+      <link name="${ns}_pan">
+     <visual>
+       <origin rpy="0 0 0" xyz="0 0 0"/>
+       <geometry>
+         <mesh filename="pan_tefal.obj"/>
+       </geometry>
+     </visual>
+     <visual name="handle">
+       <geometry>
+         <cylinder radius="0.011" length="0.185"/>
+       </geometry>
+       <origin rpy="0 1.4 0" xyz="0.22 0 0.07"/>
+       <material name="stainless">
+         <color rgba="0.3 0.3 .3 1"/>
+       </material>
+     </visual>
+     <collision name="handle">
+       <geometry>
+         <cylinder radius="0.011" length="0.185"/>
+       </geometry>
+       <origin rpy="0 1.4 0" xyz="0.22 0 0.07"/>
+     </collision>
+     <collision name="bottom">
+       <geometry>
+         <cylinder radius="0.12" length="0.01"/>
+       </geometry>
+       <origin rpy="0 0 0" xyz="0 0 0.005"/>
+     </collision>
+     <collision name="collision01">
+       <geometry>
+         <mesh filename="pan_tefal-collision01.obj"/>
+       </geometry>
+       <origin rpy="0 0 0" xyz="0 0 0"/>
+     </collision>
+     <collision name="collision02">
+       <geometry>
+         <mesh filename="pan_tefal-collision02.obj"/>
+       </geometry>
+       <origin rpy="0 0 0" xyz="0 0 0"/>
+     </collision>
+     <collision name="collision03">
+       <geometry>
+         <mesh filename="pan_tefal-collision03.obj"/>
+       </geometry>
+       <origin rpy="0 0 0" xyz="0 0 0"/>
+     </collision>
+     <collision name="collision04">
+       <geometry>
+         <mesh filename="pan_tefal-collision04.obj"/>
+       </geometry>
+       <origin rpy="0 0 0" xyz="0 0 0"/>
+     </collision>
+     <collision name="collision05">
+       <geometry>
+         <mesh filename="pan_tefal-collision05.obj"/>
+       </geometry>
+       <origin rpy="0 0 0" xyz="0 0 0"/>
+     </collision>
+     <collision name="collision06">
+       <geometry>
+         <mesh filename="pan_tefal-collision06.obj"/>
+       </geometry>
+       <origin rpy="0 0 0" xyz="0 0 0"/>
+     </collision>
+     <inertial>
+       <mass value="2."/> <!-- mr^2 = 0.5*0.12^2 = 0.0072 for Z axis, lighter along other axis -->
+       <inertia ixx="0.005" iyy="0.005" izz="0.0072"/>
+     </inertial>
     </link>
-    <link name="${ns}_rightfinger">
-      <visual>
-        <origin xyz="0 0 0" rpy="0 0 ${pi}"/>
-        <geometry>
-          <mesh filename="package://franka_description/meshes/visual/finger.dae"/>
-        </geometry>
-      </visual>
-      <collision>
-        <origin xyz="0 0 0" rpy="0 0 ${pi}"/>
-        <geometry>
-          <mesh filename="package://franka_description/meshes/collision/finger.stl"/>
-        </geometry>
-      </collision>
-    </link>
-    <joint name="${ns}_finger_joint1" type="prismatic">
+    <joint name="${ns}_pan" type="fixed">
       <parent link="${ns}_hand"/>
-      <child link="${ns}_leftfinger"/>
+      <child link="${ns}_pan"/>
       <origin xyz="0 0 0.0584" rpy="0 0 0"/>
-      <axis xyz="0 1 0"/>
-      <limit effort="20" lower="0.0" upper="0.04" velocity="0.2"/>
-    </joint>
-    <joint name="${ns}_finger_joint2" type="prismatic">
-      <parent link="${ns}_hand"/>
-      <child link="${ns}_rightfinger"/>
-      <origin xyz="0 0 0.0584" rpy="0 0 0"/>
-      <axis xyz="0 -1 0"/>
-      <limit effort="20" lower="0.0" upper="0.04" velocity="0.2"/>
-      <mimic joint="${ns}_finger_joint1" />
     </joint>
   </xacro:macro>

File: CS141 Final Project/Panda_Juggling/resources/franka_description/robots/pan.xacro (robot description, xacro)
@@ -1,21 +1,15 @@
-<?xml version="1.0" ?>
-<!-- =================================================================================== -->
-<!-- |    This document was autogenerated by xacro from hand.urdf.xacro                | -->
-<!-- |    EDITING THIS FILE BY HAND IS NOT RECOMMENDED                                 | -->
-<!-- =================================================================================== -->
-<robot name="hand">
-  <link name="panda_hand">
-    <visual>
-      <geometry>
-        <mesh filename="package://franka_description/meshes/visual/hand.dae"/>
-      </geometry>
-    </visual>
-    <collision>
-      <geometry>
-        <mesh filename="package://franka_description/meshes/collision/hand.stl"/>
-      </geometry>
-    </collision>
-  </link>
-  <link name="panda_pan">
+<?xml version="1.0" encoding="utf-8"?>
+<robot xmlns:xacro="http://www.ros.org/wiki/xacro" name="pan">
+  <xacro:macro name="pan" params="connected_to:='' ns:='' rpy:='0 0 0' xyz:='0 0 0' ">
+    <xacro:unless value="${connected_to == ''}">
+      <joint name="${ns}_hand_joint" type="fixed">
+        <parent link="${connected_to}"/>
+        <child link="${ns}_pan"/>
+        <origin xyz="${xyz}" rpy="${rpy}"/>
+      </joint>
+    </xacro:unless>
+  <!-- Frying pan model, Copyright (c) 2016 Oleg Klimov -->
+  <!-- LICENSE: CC-SA -->
+  <link name="${ns}_pan">
     <visual>
       <origin rpy="0 0 0" xyz="0 0 0"/>
@@ -26,5 +20,5 @@
     <visual name="handle">
       <geometry>
-        <cylinder length="0.185" radius="0.011"/>
+        <cylinder radius="0.011" length="0.185"/>
       </geometry>
       <origin rpy="0 1.4 0" xyz="0.22 0 0.07"/>
@@ -35,5 +29,5 @@
     <collision name="handle">
       <geometry>
-        <cylinder length="0.185" radius="0.011"/>
+        <cylinder radius="0.011" length="0.185"/>
       </geometry>
       <origin rpy="0 1.4 0" xyz="0.22 0 0.07"/>
@@ -41,5 +35,5 @@
     <collision name="bottom">
       <geometry>
-        <cylinder length="0.01" radius="0.12"/>
+        <cylinder radius="0.12" length="0.01"/>
       </geometry>
       <origin rpy="0 0 0" xyz="0 0 0.005"/>
@@ -82,13 +76,8 @@
     </collision>
     <inertial>
-      <mass value="2."/>
-      <!-- mr^2 = 0.5*0.12^2 = 0.0072 for Z axis, lighter along other axis -->
+      <mass value="2."/> <!-- mr^2 = 0.5*0.12^2 = 0.0072 for Z axis, lighter along other axis -->
       <inertia ixx="0.005" iyy="0.005" izz="0.0072"/>
     </inertial>
   </link>
-  <joint name="panda_pan" type="fixed">
-    <parent link="panda_hand"/>
-    <child link="panda_pan"/>
-    <origin rpy="0 0 0" xyz="0 0 0.0584"/>
-  </joint>
+  </xacro:macro>
 </robot>

File: CS141 Final Project/Panda_Juggling/resources/franka_description/robots/pan_tefal.urdf (robot description, URDF)
Before this commit: robot hand, 2 links, 1 joints
Links:
- removed link panda_hand
- removed link panda_pan
- added link cube, mass 2.; collision cylinder length=0.01 radius=0.12; collision cylinder length=0.185 radius=0.011
Joints:
- removed joint panda_pan

File: CS141 Final Project/Panda_Juggling/resources/franka_description/robots/panda_arm_hand.urdf.xacro (robot description, xacro)
@@ -1,6 +1,6 @@
 <?xml version="1.0" encoding="utf-8"?>
 <robot xmlns:xacro="http://www.ros.org/wiki/xacro" name="panda">
-  <xacro:include filename="$(find franka_description)/robots/panda_arm.xacro"/>
-  <xacro:include filename="$(find franka_description)/robots/hand.xacro"/>
+  <xacro:include filename="/home/sharan/catkin_ws/src/probrob/pybullet-planning/models/franka_description/robots/panda_arm.xacro"/>
+  <xacro:include filename="/home/sharan/catkin_ws/src/probrob/pybullet-planning/models/franka_description/robots/hand.xacro"/>
   <xacro:panda_arm />
   <xacro:hand ns="panda" rpy="0 0 ${-pi/4}" connected_to="panda_link8"/>

File: CS141 Final Project/Panda_Juggling/resources/franka_description/robots/panda_arm_hand_edit.urdf (robot description, URDF)
Before this commit: robot panda, 11 links, 10 joints
Links:
- removed link panda_pan
- added link panda_leftfinger; collision mesh filename=package://franka_description/meshes/collision/finger.stl; visual mesh filename=package://franka_description/meshes/visual/finger.dae
- added link panda_rightfinger; collision mesh filename=package://franka_description/meshes/collision/finger.stl; visual mesh filename=package://franka_description/meshes/visual/finger.dae
- added link tool_link
Joints:
- removed joint panda_pan
- added joint panda_finger_joint1: type prismatic, parent panda_hand, child panda_leftfinger, origin xyz=0 0 0.0584 rpy=0 0 0, axis 0 1 0, limit lower=0.0 upper=0.04 effort=20 velocity=0.2
- added joint panda_finger_joint2: type prismatic, parent panda_hand, child panda_rightfinger, origin xyz=0 0 0.0584 rpy=0 0 0, axis 0 -1 0, limit lower=0.0 upper=0.04 effort=20 velocity=0.2, mimic joint=panda_finger_joint1
- added joint tool_joint: type fixed, parent panda_link8, child tool_link, origin xyz=0.0 0 0.1 rpy=0 0 2.35619449019, axis 0 0 1
- joint panda_hand_joint: origin xyz=0 0 0 rpy=0 0 -0.7853981633974483 -> xyz=0 0 0 rpy=0 0 -0.785398163397
- joint panda_joint2: origin xyz=0 0 0 rpy=-1.5707963267948966 0 0 -> xyz=0 0 0 rpy=-1.57079632679 0 0
- joint panda_joint3: origin xyz=0 -0.316 0 rpy=1.5707963267948966 0 0 -> xyz=0 -0.316 0 rpy=1.57079632679 0 0
- joint panda_joint4: origin xyz=0.0825 0 0 rpy=1.5707963267948966 0 0 -> xyz=0.0825 0 0 rpy=1.57079632679 0 0
- joint panda_joint5: origin xyz=-0.0825 0.384 0 rpy=-1.5707963267948966 0 0 -> xyz=-0.0825 0.384 0 rpy=-1.57079632679 0 0
- joint panda_joint6: origin xyz=0 0 0 rpy=1.5707963267948966 0 0 -> xyz=0 0 0 rpy=1.57079632679 0 0
- joint panda_joint7: origin xyz=0.088 0 0 rpy=1.5707963267948966 0 0 -> xyz=0.088 0 0 rpy=1.57079632679 0 0

File: CS141 Final Project/Panda_Juggling/resources/franka_description/robots/panda_arm_hand_pan.urdf (robot description, URDF)
Before this commit: robot panda, 11 links, 10 joints
Links:
- removed link panda_pan
- added link _pan, mass 2.; collision cylinder length=0.01 radius=0.12; collision cylinder length=0.185 radius=0.011
- added link pan_pan, mass 2.; collision cylinder length=0.01 radius=0.12; collision cylinder length=0.185 radius=0.011
- added link panda_leftfinger; collision mesh filename=package://franka_description/meshes/collision/finger.stl; visual mesh filename=package://franka_description/meshes/visual/finger.dae
- added link panda_rightfinger; collision mesh filename=package://franka_description/meshes/collision/finger.stl; visual mesh filename=package://franka_description/meshes/visual/finger.dae
Joints:
- removed joint panda_pan
- added joint pan_hand_joint: type fixed, parent panda_hand, child pan_pan, origin xyz=0 0 0 rpy=0 0 1
- added joint panda_finger_joint1: type prismatic, parent panda_hand, child panda_leftfinger, origin xyz=0 0 0.0584 rpy=0 0 0, axis 0 1 0, limit lower=0.0 upper=0.04 effort=20 velocity=0.2
- added joint panda_finger_joint2: type prismatic, parent panda_hand, child panda_rightfinger, origin xyz=0 0 0.0584 rpy=0 0 0, axis 0 -1 0, limit lower=0.0 upper=0.04 effort=20 velocity=0.2, mimic joint=panda_finger_joint1
