Commit message: tuning parameters and rewards

File: CS141 Final Project/Panda_Juggling/resources/franka_description/robots/panda_arm_hand.urdf (robot description, URDF)
Before this commit: robot panda, 11 links, 10 joints
Links:
- link panda_pan: geometry collision cylinder length=0.01 radius=0.12; collision mesh filename=pan_tefal-collision01.obj

Commit message: wroking base version

File: CS141 Final Project/Panda_Juggling/resources/franka_description/robots/panda_arm_hand.urdf (robot description, URDF)
Before this commit: robot panda, 11 links, 10 joints
Joints:
- joint panda_pan: origin xyz=0 0 0.06 rpy=0 0 0 -> xyz=0 0 0.07 rpy=0 0 0
